Commit message: attach lidar sensor to rcj_robot

File: rcj_robot/urdf/rcj_robot.urdf (robot description, URDF)
Before this commit: robot rcj_robot, 3 links, 2 joints
Links:
- removed link head_link
- added link lidar_link; visual cylinder length=0.04 radius=0.03
- link body_link: geometry collision cylinder length=0.11 radius=0.11; visual cylinder length=0.11 radius=0.11
Joints:
- removed joint head_joint
- added joint lidar_joint: type fixed, parent base_link, child lidar_link, origin xyz=0 0 0.13 rpy=0 0 0
- joint body_joint: origin xyz=0 0 0.09 rpy=0 0 0 -> xyz=0 0 0.055 rpy=0 0 0
